File: Project/eurovISOn.kicad_sch (KiCad schematic)
At the start: 43 parts, among them IC1 W25Q16JVUXIQ, J1 USB_C_Receptacle_USB2.0, J2 JST SH, J3 Pico EZmate, J4 SWD, SW1 boot, SW2 SW_Push, U1 74AHCT1G125, U2 USBLC6-2SC6, U3 RP2040, U4 XC6206PxxxMR-Regulator_Linear, Y1 12MHz

Commit message: final revision
Parts:
- removed J4: SWD, PCM_marbastlib-various:CON_TC2030_outlined, symbol Connector_Generic:Conn_01x05
- added J5: TC2030_SWD, PCM_marbastlib-various:CON_TC2030_outlined, symbol PCM_marbastlib-various:TC2030_SWD
- F1, J1, R2, R3, U2: now not fitted; now left out of the parts list
Connections:
- net GPIO0 is gone; now on net RGB MCU: U3.2 (GPIO0)
- net +3V3: now also J5.1 (VCC)
- net GND: now also J5.5 (GND)
- net RGB MCU: no longer U3.3 (GPIO1)
- net SWCLK: now also J5.4 (SWCLK)
- net SWD: now also J5.2 (SWDIO)
- net ~{RESET}: now also J5.3 (~{RST})
- new net GPIO1: U3.3 (GPIO1)
- no-connect marks 3 -> 4
Other:
- note added: "(removed from board in favour of DB)"
- note added: "Programming header"
- note removed: "Maybe add something on shield?"
- note removed: "W25Q16JVUXIQ"
- moved on the sheet: C18, IC1, R7, R9, SW1, SW2
