File: Project/plate.kicad_pcb (KiCad board)
At the start: 2 copper layers, 271.5 x 97.7 mm, 2 parts

Commit message: final revision
Other:
- outline, holes or cut-outs redrawn
Changed lines of the file:
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@@
+		(layer "Edge.Cuts")
+	)
+	(gr_circle
+		(center 148.43125 14.2125)
+		(end 149.68125 14.2125)
+		(stroke
+			(width 0.2)
+			(type default)
+		)
+		(fill none)
 		(layer "Edge.Cuts")
 	)
@@
 		(start 257.825 62.85)
 		(end 243.825 62.85)
+		(stroke
+			(width 0.2)
+			(type default)
+		)
+		(layer "Edge.Cuts")
+	)
+	(gr_line
+		(start 261.347372 17.4625)
+		(end 160.746508 17.5375)
 		(stroke
 			(width 0.2)
@@
 		(layer "Edge.Cuts")
 	)
+	(gr_arc
+		(start 154.007505 108.329011)
+		(mid 153.139669 108.90887)
+		(end 152.115994 109.1125)
+		(stroke
+			(width 0.2)
+			(type default)
+		)
+		(layer "Edge.Cuts")
+	)
 	(gr_line
 		(start 219.725 76.85)
@@
 		(layer "Edge.Cuts")
 	)
+	(gr_arc
+		(start 160.746508 17.5375)
+		(mid 159.332681 17.220268)
+		(end 158.147889 16.386117)
+		(stroke
+			(width 0.2)
+			(type default)
+		)
+		(layer "Edge.Cuts")
+	)
+	(gr_arc
+		(start 142.854995 12.245989)
+		(mid 143.722831 11.66613)
+		(end 144.746506 11.4625)
+		(stroke
+			(width 0.2)
+			(type default)
+		)
+		(layer "Edge.Cuts")
+	)
 	(gr_line
 		(start 210.2 43.8)
@@
 		(layer "Edge.Cuts")
 	)
+	(gr_arc
+		(start 158.147632 104.188884)
+		(mid 159.347343 103.429732)
+		(end 160.746251 103.1875)
+		(stroke
+			(width 0.2)
+			(type default)
+		)
+		(layer "Edge.Cuts")
+	)
 	(gr_line
 		(start 35.515127 103.1875)
-		(end 261.34737 103.1875)
+		(end 136.115992 103.1875)
 		(stroke
 			(width 0.2)
@@
 	(gr_arc
 		(start 35.51513 17.4625)
-		(mid 34.108768 17.182757)
+		(mid 34.108767 17.182758)
 		(end 32.916511 16.386117)
 		(stroke
@@
 		(layer "Edge.Cuts")
 	)
+	(gr_circle
+		(center 148.43125 106.4375)
+		(end 149.68125 106.4375)
+		(stroke
+			(width 0.2)
+			(type default)
+		)
+		(fill none)
+		(layer "Edge.Cuts")
+	)
 	(gr_arc
 		(start 12.7 18.277628)
@@
 	)
 	(gr_line
+		(start 152.115994 109.1125)
+		(end 144.74625 109.1125)
+		(stroke
+			(width 0.2)
+			(type default)
+		)
+		(layer "Edge.Cuts")
+	)
+	(gr_line
+		(start 144.746506 11.4625)
+		(end 152.11625 11.4625)
+		(stroke
+			(width 0.2)
+			(type default)
+		)
+		(layer "Edge.Cuts")
+	)
+	(gr_line
 		(start 110.1875 38.75)
 		(end 110.1875 24.75)
@@
 	)
 	(gr_line
+		(start 142.854738 108.32901)
+		(end 138.714611 104.188883)
+		(stroke
+			(width 0.2)
+			(type default)
+		)
+		(layer "Edge.Cuts")
+	)
+	(gr_line
 		(start 279.25625 21.0745)
 		(end 264.25625 21.0745)
@@
 		(start 243.825 62.85)
 		(end 243.825 76.85)
+		(stroke
+			(width 0.2)
+			(type default)
+		)
+		(layer "Edge.Cuts")
+	)
+	(gr_line
+		(start 138.714868 16.386116)
+		(end 142.854995 12.245989)
 		(stroke
 			(width 0.2)
@@
 	)
 	(gr_line
+		(start 160.746251 103.1875)
+		(end 261.34737 103.1875)
+		(stroke
+			(width 0.2)
+			(type default)
+		)
+		(layer "Edge.Cuts")
+	)
+	(gr_line
 		(start 91.1375 24.75)
 		(end 77.1375 24.75)
@@
 	)
 	(gr_line
-		(start 261.347372 17.4625)
+		(start 136.116249 17.462499)
 		(end 35.51513 17.4625)
 		(stroke
@@
 		(layer "Edge.Cuts")
 	)
+	(gr_arc
+		(start 152.11625 11.4625)
+		(mid 153.139933 11.666112)
+		(end 154.007762 12.24599)
+		(stroke
+			(width 0.2)
+			(type default)
+		)
+		(layer "Edge.Cuts")
+	)
+	(gr_arc
+		(start 144.74625 109.1125)
+		(mid 143.722567 108.908888)
+		(end 142.854738 108.32901)
+		(stroke
+			(width 0.2)
+			(type default)
+		)
+		(layer "Edge.Cuts")
+	)
 	(gr_line
 		(start 215.25 43.8)
@@
 	)
 	(gr_line
+		(start 154.007762 12.24599)
+		(end 158.147889 16.386117)
+		(stroke
+			(width 0.2)
+			(type default)
+		)
+		(layer "Edge.Cuts")
+	)
+	(gr_line
 		(start 224.775 62.85)
 		(end 224.775 76.85)
@@
 		(start 172.1 43.8)
 		(end 158.1 43.8)
+		(stroke
+			(width 0.2)
+			(type default)
+		)
+		(layer "Edge.Cuts")
+	)
+	(gr_arc
+		(start 136.115992 103.1875)
+		(mid 137.514899 103.429732)
+		(end 138.714611 104.188883)
 		(stroke
 			(width 0.2)
@@
 		(layer "Edge.Cuts")
 	)
+	(gr_arc
+		(start 138.714868 16.386116)
+		(mid 137.522616 17.182767)
+		(end 136.116249 17.462499)
+		(stroke
+			(width 0.2)
+			(type default)
+		)
+		(layer "Edge.Cuts")
+	)
 	(gr_line
 		(start 89.04375 100.6625)
@@
 	(gr_arc
 		(start 32.948624 104.232162)
-		(mid 34.129645 103.458677)
+		(mid 34.129647 103.458679)
 		(end 35.515127 103.1875)
 		(stroke
@@
 		(stroke
 			(width 0.2)
+			(type default)
+		)
+		(layer "Edge.Cuts")
+	)
+	(gr_line
+		(start 158.147632 104.188884)
+		(end 154.007505 108.329011)
+		(stroke
+			(width 0.2)
