File: Project/rgb.kicad_sch (KiCad schematic)
At the start: 10 parts

Commit message: update
Parts:
- added LED11, LED12, LED13, LED14: SK6812MINI-E, PCM_marbastlib-various:LED_6028R, symbol PCM_marbastlib-various:SK6812MINI-E
Connections:
- net +5V: now also LED11.1 (VDD), LED12.1 (VDD), LED13.1 (VDD), LED14.1 (VDD)
- net GND: now also LED11.4 (VSS), LED12.4 (VSS), LED13.4 (VSS), LED14.4 (VSS)
- net at LED4.3 (DIN): now also LED12.2 (DOUT); no longer LED3.2 (DOUT)
- net at LED9.3 (DIN): now also LED13.2 (DOUT); no longer LED8.2 (DOUT)
- net at LED6.3 (DIN): now also LED14.2 (DOUT); no longer LED5.2 (DOUT)
- new net: LED11.2 (DOUT), LED12.3 (DIN)
- new net: LED11.3 (DIN), LED3.2 (DOUT)
- new net: LED14.3 (DIN), LED5.2 (DOUT)
- new net: LED13.3 (DIN), LED8.2 (DOUT)
Other:
- moved on the sheet: LED10, LED4, LED5, LED6, LED7, LED8, LED9
